Commit message: Refactors icarus_bringup to icarus_description

File: src/icarus_description/urdf/icarus.urdf.xacro (robot description, xacro)
@@ -41,5 +41,5 @@
         </visual>
     </link>
-    <joint name="base_to_link1" type="revolute">
+    <joint name="joint1" type="revolute">
         <axis xyz="0 0 1" rpy="0 0 ${M_PI}"/>
         <limit effort="1000.0" lower="${-M_PI/2}" upper="${M_PI/2}" velocity="0.5" />
@@ -57,8 +57,8 @@
         </visual>
     </link>
-    <joint name="link1_to_link2" type="revolute">
-        <axis xyz="0 1 0" />
+    <joint name="joint2" type="revolute">
+        <axis xyz="0 -1 0" />
         <limit effort="1000.0" lower="${-3/4*M_PI}" upper="${3/4*M_PI}" velocity="0.5" />
-        <origin xyz="0 0 ${link1_length}" />
+        <origin xyz="0 0 ${link1_length}" rpy="0 ${M_PI/2} 0"/>
         <parent link="link1" />
         <child link="link2" />
@@ -73,6 +73,6 @@
         </visual>
     </link>
-    <joint name="link2_to_link3" type="revolute">
-        <axis xyz="0 1 0" />
+    <joint name="joint3" type="revolute">
+        <axis xyz="0 -1 0" />
         <limit effort="1000.0" lower="${-3/4*M_PI}" upper="${3/4*M_PI}" velocity="0.5" />
         <origin xyz="0 0 ${link2_length}" />
@@ -124,5 +124,5 @@
             <origin xyz="0 0 0" rpy="0 0 ${M_PI/2}"/>
             <geometry>
-                <mesh filename="package://icarus_bringup/urdf/meshes/kinect.dae"/>
+                <mesh filename="package://icarus_description/urdf/meshes/kinect.dae"/>
             </geometry>
         </visual>

Commit message: Updates the definition for new semipermanent setup

File: src/icarus_description/urdf/icarus.urdf.xacro (robot description, xacro)
@@ -3,4 +3,6 @@
     <xacro:property name="M_PI" value="3.14159" />
     <!-- Robot Params -->
+    <xacro:property name="base_xyz" value="-0.2794 0.2111375 0" />
+    <xacro:property name="base_rpy" value="0 0 -0.523599"/>
     <xacro:property name="base_width" value="0.04" />
     <xacro:property name="base_height" value="0.17" />
@@ -13,9 +15,9 @@
       <xacro:property name="cam_py" value="-0.25" />
       <xacro:property name="cam_pz" value="0.4" />-->
-    <xacro:property name="cam_px" value="-1.8" />
-    <xacro:property name="cam_py" value="-0.35" />
-    <xacro:property name="cam_pz" value="0.2" />
+    <xacro:property name="cam_px" value="-1.5" />
+    <xacro:property name="cam_py" value="-0.3794125" />
+    <xacro:property name="cam_pz" value="0.384175" />
     <xacro:property name="cam_or" value="0.0" />
-    <xacro:property name="cam_op" value="${5.0*M_PI/180}" />
+    <xacro:property name="cam_op" value="${10.0*M_PI/180}" />
     <xacro:property name="cam_oy" value="0.244" />
     <xacro:property name="kinect_height" value="0.073" />
@@ -23,5 +25,5 @@
     <xacro:property name="table_thickness" value="0.05" />
     <xacro:property name="table_length" value="2.5" />
-    <xacro:property name="table_width" value="1.0" />
+    <xacro:property name="table_width" value="0.911225" />
     <!-- Macros -->
     <xacro:macro name="material_color" params="name rgba">
@@ -31,4 +33,11 @@
     </xacro:macro>
     <xacro:material_color name="default" rgba="0.7 0.7 0.7 1.0" />
+    <!-- World -->
+    <link name="world" />
+    <joint name="world_to_base" type="fixed">
+        <origin xyz="${base_xyz}" rpy="${base_rpy}"/>
+        <parent link="world"/>
+        <child link="base_link" />
+    </joint>
     <!-- Robot Arm -->
     <link name="base_link">
@@ -103,7 +112,7 @@
     </link>
     <!-- Kinect -->
-    <joint name="base_to_kinect" type="fixed">
+    <joint name="world_to_kinect" type="fixed">
         <origin xyz="${cam_px} ${cam_py} ${cam_pz}" rpy="${cam_or} ${cam_op} ${cam_oy}"/>
-        <parent link="base_link"/>
+        <parent link="world"/>
         <child link="kinect" />
     </joint>
@@ -142,7 +151,7 @@
     </link>
     <!-- Table -->
-    <joint name="base_to_table" type="fixed">
+    <joint name="world_to_table" type="fixed">
         <origin xyz="0 0 0" />
-        <parent link="base_link" />
+        <parent link="world" />
         <child link="table" />
     </joint>
@@ -158,7 +167,7 @@
         </visual>
     </link>
-    <joint name="base_to_support" type="fixed">
+    <joint name="world_to_support" type="fixed">
         <origin xyz="${cam_px} ${cam_py} ${cam_pz/2-kinect_height/4}" />
-        <parent link="base_link" />
+        <parent link="world" />
         <child link="support" />
     </joint>

Commit message: Updates the link lengths

File: src/icarus_description/urdf/icarus.urdf.xacro (robot description, xacro)
@@ -8,7 +8,7 @@
     <xacro:property name="base_height" value="0.17" />
     <xacro:property name="link_radius" value="0.015" />
-    <xacro:property name="link1_length" value="0.05" />
+    <xacro:property name="link1_length" value="${0.245-base_height}" />
     <xacro:property name="link2_length" value="0.22" />
-    <xacro:property name="link3_length" value="0.22" />
+    <xacro:property name="link3_length" value="0.24" />
     <!-- Kinect Params -->
     <!--  <xacro:property name="cam_px" value="-1.2" />

Commit message: Updates location of the robot back to center

File: src/icarus_description/urdf/icarus.urdf.xacro (robot description, xacro)
@@ -3,4 +3,23 @@
     <xacro:property name="M_PI" value="3.14159" />
     <!-- Robot Params -->
+    <xacro:property name="base_xyz" value="-0.3 0 0" />
+    <xacro:property name="base_rpy" value="0 0 0"/>
+    <xacro:property name="base_width" value="0.025" />
+    <xacro:property name="base_height" value="0.13" />
+    <xacro:property name="link_radius" value="0.015" />
+    <xacro:property name="link1_length" value="${0.24-base_height}" />
+    <xacro:property name="link2_length" value="0.22" />
+    <xacro:property name="link3_length" value="0.24" />
+    <!-- Workspace for visualization only -->
+    <xacro:property name="xlim_l" value="-0.2"/>
+    <xacro:property name="xlim_u" value="0.05"/>
+    <xacro:property name="ylim_l" value="-0.2"/>
+    <xacro:property name="ylim_u" value="0.2"/>
+    <xacro:property name="zlim_l" value="0.05"/>
+    <xacro:property name="zlim_u" value="0.3"/>
+    <xacro:property name="xlim" value="${xlim_u-xlim_l}" />
+    <xacro:property name="ylim" value="${ylim_u-ylim_l}" />
+    <xacro:property name="zlim" value="${zlim_u-zlim_l}" />
+<!-- old - clamp rotated 30 deg
     <xacro:property name="base_xyz" value="-0.2794 0.2111375 0" />
     <xacro:property name="base_rpy" value="0 0 -0.523599"/>
@@ -11,4 +30,5 @@
     <xacro:property name="link2_length" value="0.22" />
     <xacro:property name="link3_length" value="0.24" />
+-->
     <!-- Kinect Params -->
     <!--  <xacro:property name="cam_px" value="-1.2" />
@@ -183,3 +203,18 @@
         </visual>
     </link>
+    <joint name="world_to_workspace" type="fixed" >
+        <parent link="world"/>
+        <child link="workspace"/>
+    </joint>
+    <link name="workspace" >
+        <visual>
+            <origin xyz="${xlim_l+xlim/2} ${ylim_l+ylim/2} ${zlim_l+zlim/2}" />
+            <geometry>
+                <box size="${xlim} ${ylim} ${zlim}" />
+            </geometry>
+            <material name="red_trans">
+                <color rgba="1 0 0 0.3" />
+            </material>
+        </visual>
+    </link>
 </robot>

Commit message: Fixes camera support base

File: src/icarus_description/urdf/icarus.urdf.xacro (robot description, xacro)
@@ -196,5 +196,5 @@
             <origin xyz="0 0 0" />
             <geometry>
-                <box size="0.2 0.3 ${cam_pz-kinect_height/2}"/>
+                <box size="0.15 0.15 ${cam_pz-kinect_height/2}"/>
             </geometry>
             <material name="blue">
